File: PCB_Design_Kicad/MIDIFAM.kicad_sch (KiCad schematic)
At the start: 57 parts, among them IC1 DAC8562SDGSR, J1 PWR_IN, J10 midi, J11 back bottom, J13 back top, J2 ISP connector, U1 LM7805_TO220, U4 OPA4196xD, U5 6N137, U6 ATmega328-A

Commit message: more bom
Parts:
- C1, C10, C12, C14, C2, C3: LCSC C143639 -> C14663
- C13: LCSC C2691405 -> C14663
- R20, R22: value 6k -> 33k; LCSC (none) -> C4216
- R21, R23: value 10k -> 56k; LCSC C845630 -> C23206
- U1: footprint Package_TO_SOT_THT:TO-220-3_Vertical -> Package_TO_SOT_THT:TO-220-3_Horizontal_TabUp
Other:
- moved on the sheet: R20, R22
Changed lines of the file:
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@@
 	(wire
 		(pts
-			(xy 127 73.66) (xy 132.08 73.66)
+			(xy 127 73.66) (xy 134.62 73.66)
 		)
 		(stroke
@@
 	(wire
 		(pts
-			(xy 137.16 73.66) (xy 142.24 73.66)
+			(xy 139.7 73.66) (xy 142.24 73.66)
 		)
 		(stroke
@@
 	(wire
 		(pts
-			(xy 137.16 39.37) (xy 142.24 39.37)
+			(xy 139.7 39.37) (xy 142.24 39.37)
 		)
 		(stroke
@@
 	(wire
 		(pts
-			(xy 127 39.37) (xy 132.08 39.37)
+			(xy 127 39.37) (xy 134.62 39.37)
 		)
 		(stroke
@@
 			)
 		)
-		(property "LCSC" "C2691405"
+		(property "LCSC" "C14663"
 			(at 255.905 151.13 0)
 			(effects
@@
 			)
 		)
-		(property "LCSC" "C143639"
+		(property "LCSC" "C14663"
 			(at 23.495 34.925 0)
 			(effects
@@
 			)
 		)
-		(property "LCSC" "C143639"
+		(property "LCSC" "C14663"
 			(at 229.87 135.89 0)
 			(effects
@@
 			)
 		)
-		(property "LCSC" "C143639"
+		(property "LCSC" "C14663"
 			(at 80.01 165.735 0)
 			(effects
@@
 			)
 		)
-		(property "LCSC" "C143639"
+		(property "LCSC" "C14663"
 			(at 229.87 146.685 0)
 			(effects
@@
 		(dnp no)
 		(property "Reference" "R23"
-			(at 130.81 80.645 0)
+			(at 130.175 76.2 0)
 			(effects
 				(font
@@
 			)
 		)
-		(property "Value" "10k"
-			(at 130.81 78.74 0)
+		(property "Value" "56k"
+			(at 130.175 78.105 0)
 			(effects
 				(font
@@
 			)
 		)
-		(property "LCSC" "C845630"
+		(property "LCSC" "C23206"
 			(at 127 77.47 0)
 			(effects
@@
 			)
 		)
-		(property "LCSC" "C143639"
+		(property "LCSC" "C14663"
 			(at 48.26 23.495 0)
 			(effects
@@
 			)
 		)
-		(property "LCSC" "C143639"
+		(property "LCSC" "C14663"
 			(at 36.83 23.495 0)
 			(effects
@@
 	(symbol
 		(lib_id "Device:R_Small")
-		(at 134.62 39.37 270)
+		(at 137.16 39.37 270)
 		(unit 1)
 		(exclude_from_sim no)
@@
 		(dnp no)
 		(property "Reference" "R20"
-			(at 137.795 43.815 90)
+			(at 137.16 41.91 90)
 			(effects
 				(font
@@
 			)
 		)
-		(property "Value" "6k"
-			(at 137.795 41.91 90)
+		(property "Value" "33k"
+			(at 137.16 43.815 90)
 			(effects
 				(font
@@
 		)
 		(property "Footprint" "Resistor_SMD:R_0603_1608Metric_Pad0.98x0.95mm_HandSolder"
-			(at 134.62 39.37 0)
+			(at 137.16 39.37 0)
 			(effects
 				(font
@@
 		)
 		(property "Datasheet" "~"
-			(at 134.62 39.37 0)
+			(at 137.16 39.37 0)
 			(effects
 				(font
@@
 		)
 		(property "Description" "Resistor, small symbol"
-			(at 134.62 39.37 0)
+			(at 137.16 39.37 0)
 			(effects
 				(font
@@
 			)
 		)
-		(property "LCSC" ""
-			(at 134.62 39.37 0)
+		(property "LCSC" "C4216"
+			(at 137.16 39.37 0)
 			(effects
 				(font
@@
 		)
 		(property "Price (single)" ""
-			(at 134.62 39.37 0)
+			(at 137.16 39.37 0)
 			(effects
 				(font
@@
 			)
 		)
-		(property "Footprint" "Package_TO_SOT_THT:TO-220-3_Vertical"
+		(property "Footprint" "Package_TO_SOT_THT:TO-220-3_Horizontal_TabUp"
 			(at 261.62 140.97 0)
 			(effects
@@
 		(dnp no)
 		(property "Reference" "R21"
-			(at 130.175 46.355 0)
+			(at 130.175 42.545 0)
 			(effects
 				(font
@@
 			)
 		)
-		(property "Value" "10k"
+		(property "Value" "56k"
 			(at 130.175 44.45 0)
 			(effects
@@
 			)
 		)
-		(property "LCSC" "C845630"
+		(property "LCSC" "C23206"
 			(at 127 43.18 0)
 			(effects
@@
 	(symbol
 		(lib_id "Device:R_Small")
-		(at 134.62 73.66 270)
+		(at 137.16 73.66 270)
 		(unit 1)
 		(exclude_from_sim no)
@@
 		(on_board yes)
 		(dnp no)
-		(fields_autoplaced yes)
 		(property "Reference" "R22"
-			(at 137.795 77.47 90)
+			(at 137.16 76.2 90)
 			(effects
 				(font
@@
 			)
 		)
-		(property "Value" "6k"
-			(at 137.795 75.565 90)
+		(property "Value" "33k"
+			(at 137.16 78.74 90)
 			(effects
 				(font
@@
 		)
 		(property "Footprint" "Resistor_SMD:R_0603_1608Metric_Pad0.98x0.95mm_HandSolder"
-			(at 134.62 73.66 0)
+			(at 137.16 73.66 0)
 			(effects
 				(font
@@
 		)
 		(property "Datasheet" "~"
-			(at 134.62 73.66 0)
+			(at 137.16 73.66 0)
 			(effects
 				(font
@@
 		)
 		(property "Description" "Resistor, small symbol"
-			(at 134.62 73.66 0)
+			(at 137.16 73.66 0)
 			(effects
 				(font
@@
 			)
 		)
-		(property "LCSC" ""
-			(at 134.62 73.66 0)
+		(property "LCSC" "C4216"
+			(at 137.16 73.66 0)
 			(effects
 				(font
@@
 		)
 		(property "Price (single)" ""
-			(at 134.62 73.66 0)
+			(at 137.16 73.66 0)
 			(effects
 				(font

Commit message: more bom
Parts:
- C1, C10, C12, C14, C2, C3: Comment (none) -> 100n
- C11, C9: Comment (none) -> 10u; LCSC C336586 -> C263975
- C13: Comment (none) -> 0.1u
- C15, C17, C4: Comment (none) -> 1u
- C16, C5, C6, C7: Comment (none) -> 18p; LCSC C184235 -> C1647
- C18: Comment (none) -> 150n
- C8: Comment (none) -> 0.33u; LCSC C2691405 -> C1623
- D1, D7: Comment (none) -> 1N4148; LCSC C108805 -> C2128
- D5: Comment (none) -> rpp diode; LCSC C688896 -> C8598
- D6: footprint Diode_SMD:D_SOD-123 -> Diode_SMD:D_SOD-123F; Comment (none) -> rpp diode; LCSC C688896 -> C8598
- IC1: Comment (none) -> DAC8562SDGSR
- J1: Comment (none) -> PWR_IN
- J10: Comment (none) -> midi
- J11: Comment (none) -> back bottom
- J13: Comment (none) -> back top
- J2: Comment (none) -> ISP connector
- R1, R3: Comment (none) -> 240k
- R10, R14, R5, R8: Comment (none) -> 220R; LCSC C365121 -> C22962
- R11, R12, R13, R15, R24, R6, R9: Comment (none) -> 10k; LCSC C845630 -> C25804
- R16, R17, R2, R4: Comment (none) -> 47k; LCSC C2907042 -> C25819
- R18, R19, R7: Comment (none) -> 1k; LCSC C2758735 -> C21190
- R20, R22: Comment (none) -> 33k
- R21, R23: Comment (none) -> 56k
- U1: Comment (none) -> LM7805_TO220
- U4: Comment (none) -> OPA4196xD
- U5: Comment (none) -> 6N137
- U6: Comment (none) -> ATmega328-A
- xtal1: Comment (none) -> 16MHz
