File: PCB_Design_Kicad/MIDIFAM.kicad_sch (KiCad schematic)
At the start: 57 parts, among them IC1 DAC8562SDGSR, J1 PWR_IN, J10 midi, J11 back bottom, J13 back top, J2 ISP connector, U1 LM7805_TO220, U4 OPA4196xD, U5 6N137, U6 ATmega328-A

Commit message: pcb
Parts:
- added J17, J18: Conn_01x07, Connector_PinHeader_2.54mm:PinHeader_1x07_P2.54mm_Vertical, symbol Connector_Generic:Conn_01x07
- added U2: OPA4196xD, Package_SO:TSSOP-14_4.4x5mm_P0.65mm, symbol Amplifier_Operational:OPA4196xD
Connections:
- new net: J18.5 (Pin_5), U2.12 (+)
- new net: J18.6 (Pin_6), U2.13 (-)
- new net: J18.7 (Pin_7), U2.14
- new net: J17.5 (Pin_5), U2.5 (+)
- new net: J17.6 (Pin_6), U2.6 (-)
- new net: J17.7 (Pin_7), U2.7
- new net: J18.3 (Pin_3), U2.10 (+)
- new net: J18.1 (Pin_1), U2.8
- new net: J18.2 (Pin_2), U2.9 (-)
- new net: J18.4 (Pin_4), U2.11 (V-)
- new net: J17.1 (Pin_1), U2.1
- new net: J17.2 (Pin_2), U2.2 (-)
- new net: J17.3 (Pin_3), U2.3 (+)
- new net: J17.4 (Pin_4), U2.4 (V+)

Commit message: pcb versions sent to jlcpcb
Parts:
- removed J17, J18: Conn_01x07, Connector_PinHeader_2.54mm:PinHeader_1x07_P2.54mm_Vertical, symbol Connector_Generic:Conn_01x07
- removed U2: OPA4196xD, Package_SO:TSSOP-14_4.4x5mm_P0.65mm, symbol Amplifier_Operational:OPA4196xD
