File: PCB_Design_Kicad/MIDIFAM.kicad_pcb (KiCad board)
At the start: 2 copper layers, 58 x 110 mm, 74 parts, among them IC1 DAC8562SDGSR, J1 PWR_IN, J10 midi, J11 back bottom, J12 front bottom, J13 back top, J14 front top, J15 SD-50BV, J16 midi, J2 ISP connector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

Commit message: more bom
Parts:
- R20, R22: value 6k -> 33k
- R21, R23: value 10k -> 56k
- U1: footprint Package_TO_SOT_THT:TO-220-3_Vertical -> Package_TO_SOT_THT:TO-220-3_Horizontal_TabUp; moved to F.Cu
- moved C15 3.04 mm to (90.9, 62.1)
- moved R6 3.04 mm to (93.2, 62.4)
- moved D5 1.25 mm to (92.8, 33.2)
- moved U1 0.77 mm to (87.4, 40.0)
Routing:
- net Net-(U4A-+): track 21.2 -> 25.9 mm
- net /pwm_vel_A: track 12.6 -> 9.15 mm
- net /IO Control PCB/adv_clock_f: track 77.1 -> 78.4 mm
- net /IO Control PCB/led_b1_f: track 50.5 -> 49.4 mm
- net Net-(U4B--): track 5.78 -> 5.00 mm
- net /IO Control PCB/led_b2_f: track 50.8 -> 50.0 mm
- net Net-(U4A--): track 4.87 -> 4.17 mm
- net Net-(J16-Pin_2): track 18.5 -> 17.9 mm
- net /IO Control PCB/voct_a_f: track 39.1 -> 38.5 mm
- net /MISO: track 7.94 -> 7.42 mm
Other:
- board text added: "K"

Commit message: more bom
Parts:
- D6: footprint Diode_SMD:D_SOD-123 -> Diode_SMD:D_SOD-123F
- J15: footprint SamacSys_Parts:SD-50BV -> WeirdVibes_Eurorack:CUI SD-50BV MIDI DIN-5
- moved SW3 1.77 mm to (61.3, 101.0)
- moved C15 1.41 mm to (91.6, 63.4)
- moved R6 1.08 mm to (93.6, 63.4)
- moved C4 0.40 mm to (86.8, 64.4)
- moved R9 0.40 mm to (88.3, 64.4)
- moved D4 0.27 mm to (70.5, 103.5)
Routing:
- net Net-(U4A-+): track 25.9 -> 24.2 mm
- net Net-(J16-Pin_2): track 17.9 -> 17.0 mm
- net Net-(J16-Pin_3): track 14.3 -> 13.6 mm
- net /pwm_vel_A: track 9.15 -> 8.50 mm
- net Net-(U4B-+): track 28.6 -> 29.2 mm
Other:
- board size 58 x 110 mm -> 58 x 90.6 mm

Commit message: pcb
Parts:
- added IC2: DAC8562SDGSR, SamacSys_Parts:SOP50P490X110-10N, F.Cu at (115.9, 130.3)
- added J17: Conn_01x07, Connector_PinHeader_2.54mm:PinHeader_1x07_P2.54mm_Vertical, B.Cu at (112.1, 101.8)
- added J18: Conn_01x07, Connector_PinHeader_2.54mm:PinHeader_1x07_P2.54mm_Vertical, B.Cu at (119.6, 117.1)
- added J19: bbjack, WeirdVibes:Thonkiconn, F.Cu at (115.9, 55.1)
- added J20: Conn_01x03, Connector_PinHeader_2.54mm:PinHeader_1x03_P2.54mm_Vertical, B.Cu at (118.5, 52.0)
- added J21: Conn_01x03, Connector_PinHeader_2.54mm:PinHeader_1x03_P2.54mm_Vertical, B.Cu at (118.5, 69.8)
- added J22: bbjack, WeirdVibes:Thonkiconn, F.Cu at (115.9, 78.5)
- added J23: Conn_01x03, Connector_PinHeader_2.54mm:PinHeader_1x03_P2.54mm_Vertical, B.Cu at (118.5, 75.4)
- added J24: Conn_01x03, Connector_PinHeader_2.54mm:PinHeader_1x03_P2.54mm_Vertical, B.Cu at (118.5, 93.2)
- added U2: OPA4196xD, Package_SO:TSSOP-14_4.4x5mm_P0.65mm, F.Cu at (115.9, 109.6)
- J15: value SD-50BV -> Conn_01x05; footprint WeirdVibes_Eurorack:CUI SD-50BV MIDI DIN-5 -> Connector_PinHeader_2.54mm:PinHeader_1x05_P2.54mm_Vertical; moved to B.Cu
- J16: value midi -> Conn_01x05; footprint Connector_PinSocket_2.54mm:PinSocket_1x03_P2.54mm_Vertical -> Connector_PinHeader_2.54mm:PinHeader_1x05_P2.54mm_Vertical
- moved J15 42.8 mm to (112.0, 125.8), turned to 180 degrees
- moved J16 40.8 mm to (119.6, 125.8), turned to 180 degrees
- moved C9 25.9 mm to (83.9, 55.0)
- moved C1 25.9 mm to (90.3, 100.5)
- moved C10 25.9 mm to (90.8, 72.2)
- moved C11 25.9 mm to (106.6, 55.0)
- moved C12 25.9 mm to (104.0, 72.0)
- moved C13 25.9 mm to (88.1, 62.1)
- moved C14 25.9 mm to (105.8, 130.8)
- moved C17 25.9 mm to (96.8, 83.7)
- moved C18 25.9 mm to (96.8, 82.0)
- moved C2 25.9 mm to (106.5, 98.2)
- moved C6 25.9 mm to (91.0, 98.5)
- moved C7 25.9 mm to (91.0, 96.4)
- moved D1 25.9 mm to (89.3, 127.0)
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Connections:
- J15 pad 1: unconnected-(J15-Pad1) -> Net-(IC2-VOUTA)
- J15 pad 2: Net-(J16-Pin_3) -> Net-(IC2-VOUTB)
- J15 pad 3: unconnected-(J15-Pad3) -> Net-(IC2-GND)
- J15 pad 4: Net-(J16-Pin_2) -> Net-(IC2-~{LDAC})
- J15 pad 5: unconnected-(J15-Pad5) -> Net-(IC2-~{CLR})
- J16 pad 1: GND -> Net-(IC2-VREFIN/VREFOUT)
- J16 pad 2: Net-(J16-Pin_2) -> Net-(IC2-AVDD)
- J16 pad 3: Net-(J16-Pin_3) -> Net-(IC2-DIN)
Routing:
- net Net-(J23-Pin_1): track 0.00 -> 23.7 mm
- net Net-(J20-Pin_1): track 0.00 -> 23.7 mm
- net Net-(J23-Pin_3): track 0.00 -> 23.2 mm
- net Net-(J20-Pin_3): track 0.00 -> 22.7 mm
- net Net-(J23-Pin_2): track 0.00 -> 22.2 mm
- net Net-(J20-Pin_2): track 0.00 -> 22.2 mm
- net Net-(J16-Pin_2): track 17.0 -> 0.00 mm
- net Net-(J16-Pin_3): track 13.6 -> 0.00 mm
- net Net-(J18-Pin_7): track 0.00 -> 11.3 mm
- net Net-(J17-Pin_7): track 0.00 -> 11.2 mm, vias 0 -> 1
- net Net-(J17-Pin_1): track 0.00 -> 10.2 mm
- net Net-(IC2-~{LDAC}): track 0.00 -> 9.35 mm
- net Net-(IC2-~{CLR}): track 0.00 -> 9.07 mm
- net Net-(J18-Pin_6): track 0.00 -> 9.03 mm, vias 0 -> 1
- net Net-(J17-Pin_6): track 0.00 -> 8.88 mm, vias 0 -> 1
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Other:
- board size 58 x 90.6 mm -> 70.2 x 86.6 mm
- board text added: "10"
- board text added: "11"
- board text added: "12"
- board text added: "13"
- board text added: "14"
- board text added: "7"
- board text added: "8"
- board text added: "9"
- board text added: "gnd"
- board text added: "sw"
- board text added: "tip"

Commit message: pcb versions sent to jlcpcb
Parts:
- removed IC2: DAC8562SDGSR, SamacSys_Parts:SOP50P490X110-10N
- removed J15, J16: Conn_01x05, Connector_PinHeader_2.54mm:PinHeader_1x05_P2.54mm_Vertical
- removed J17, J18: Conn_01x07, Connector_PinHeader_2.54mm:PinHeader_1x07_P2.54mm_Vertical
- removed J19, J22: bbjack, WeirdVibes:Thonkiconn
- removed J20, J21, J23, J24: Conn_01x03, Connector_PinHeader_2.54mm:PinHeader_1x03_P2.54mm_Vertical
- removed U2: OPA4196xD, Package_SO:TSSOP-14_4.4x5mm_P0.65mm
- J3, J4, J5, J6, J7, J8: footprint WeirdVibes_Eurorack:Thonkiconn -> WeirdVibes:Thonkiconn
- J9: value adv_clock_out -> adv/clock; footprint WeirdVibes_Eurorack:Thonkiconn -> WeirdVibes:Thonkiconn
- moved J9 6.51 mm to (74.4, 123.3)
- moved J3 6.48 mm to (64.8, 83.2)
- moved J4 6.48 mm to (64.8, 94.2)
- moved J5 6.48 mm to (64.8, 105.2)
- moved J6 6.48 mm to (67.9, 83.2)
- moved J7 6.48 mm to (67.9, 94.2)
- moved J8 6.48 mm to (67.9, 105.2)
- moved D4 0.78 mm to (66.8, 129.2)
Routing:
- net Net-(J23-Pin_1): track 23.7 -> 0.00 mm
- net Net-(J20-Pin_1): track 23.7 -> 0.00 mm
- net Net-(J23-Pin_3): track 23.2 -> 0.00 mm
- net Net-(J20-Pin_3): track 22.7 -> 0.00 mm
- net Net-(J23-Pin_2): track 22.2 -> 0.00 mm
- net Net-(J20-Pin_2): track 22.2 -> 0.00 mm
- net Net-(J18-Pin_7): track 11.3 -> 0.00 mm
- net Net-(J17-Pin_7): track 11.2 -> 0.00 mm, vias 1 -> 0
- net Net-(J17-Pin_1): track 10.2 -> 0.00 mm
- net Net-(IC2-~{LDAC}): track 9.35 -> 0.00 mm
- net Net-(IC2-~{CLR}): track 9.07 -> 0.00 mm
- net Net-(J18-Pin_6): track 9.03 -> 0.00 mm, vias 1 -> 0
- net Net-(J17-Pin_6): track 8.88 -> 0.00 mm, vias 1 -> 0
- net Net-(J17-Pin_4): track 8.84 -> 0.00 mm
- net Net-(IC2-GND): track 8.24 -> 0.00 mm
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Other:
- board size 70.2 x 86.6 mm -> 58 x 86.6 mm
- board text removed: "10"
- board text removed: "11"
- board text removed: "12"
- board text removed: "13"
- board text removed: "14"
- board text removed: "7"
- board text removed: "8"
- board text removed: "9"
- board text removed: "V-CUT"
- board text removed: "gnd"
- board text removed: "sw"
- board text removed: "tip"
