File: PCB_Design_Kicad/panel/panel_MIDIFAM.kicad_pcb (KiCad board)
At the start: 2 copper layers, 193.2 x 128.5 mm, 34 parts, among them J1 CV in

Commit message: panel
Parts:
- removed J1 (x7): CV in, SamacSys_Parts:CL1384
- removed the REF** at (82.4, 58.3)
- removed the REF** at (85.1, 85.7)
- removed the REF** at (87.2, 142.3)
- removed the REF** at (83.6, 109.9)
- removed the REF** at (83.6, 119.7)
- removed the REF** at (85.1, 76.0)
- removed the REF** at (83.6, 129.4)
- removed the REF** at (93.9, 119.7)
- removed the REF** at (85.1, 95.4)
- removed the REF** at (86.9, 43.0)
- removed the REF** at (92.5, 58.6)
- removed the REF** at (93.9, 85.7)
- removed the REF** at (82.3, 49.8)
- moved REF** 13.4 mm to (128.3, 36.5), turned to 180 degrees
- moved REF** 13.3 mm to (142.8, 36.5), turned to 180 degrees
- moved REF** 12.4 mm to (135.6, 130.2)
- moved REF** 10.6 mm to (127.6, 86.6)
- moved REF** 10.2 mm to (143.6, 86.6)
- moved REF** 9.72 mm to (144.3, 111.1)
- moved REF** 9.50 mm to (127.6, 56.0)
- moved REF** 9.48 mm to (127.6, 75.5)
- moved REF** 9.32 mm to (125.8, 110.6)
- moved REF** 9.09 mm to (143.7, 56.0)
- moved REF** 9.07 mm to (143.6, 75.5)
- moved REF** 8.36 mm to (127.6, 64.5)
- moved REF** 7.88 mm to (143.6, 64.5)
- moved REF** 3.15 mm to (135.3, 110.5)
Other:
- board size 193.2 x 128.5 mm -> 30 x 128.5 mm
- board text added: "MODE"
- board text added: "learn"
- board text added: "sync"
- board text removed: "4HP"
- board text removed: "MIDI clock"
- board text removed: "Other ins/outs/controls: - MIDI clock out - {dblquote}learn{dblquote} button - mono/poly switch?"
- board text removed: "SEQ CTRL"
- board text removed: "adv/clock"
- board text removed: "learn MIDI"
- board text removed: "reset sequence"
- board text removed: "trig."
- board text removed: "velocity"

Commit message: more bom
Parts:
- moved REF** 7.75 mm to (119.9, 55.6)
- moved REF** 7.75 mm to (127.9, 129.8)
- moved REF** 7.75 mm to (136.6, 110.7)
- moved REF** 7.75 mm to (120.6, 36.1)
- moved REF** 7.75 mm to (135.1, 36.1)
- moved REF** 7.75 mm to (135.9, 75.1)
- moved REF** 7.75 mm to (136.0, 55.6)
- moved REF** 7.75 mm to (135.9, 64.1)
- moved REF** 7.75 mm to (119.9, 75.1)
- moved REF** 7.75 mm to (119.9, 64.1)
- moved REF** 7.75 mm to (135.9, 86.2)
- moved REF** 7.75 mm to (119.9, 86.2)
- moved REF** 7.48 mm to (127.9, 110.1)
- moved REF** 5.84 mm to (120.0, 110.2)
Other:
- board text added: "gate/ trig."
- board text removed: "gate/ trigger"

Commit message: pcb versions sent to jlcpcb
Parts:
- added REF**: Mounting_Hole_Jack, WeirdVibes_Eurorack:Mounting_Hole_Jack, F.Cu at (113.3, 110.7)
- added REF**: MountingHole_3.2mm_M3, MountingHole:MountingHole_3.2mm_M3, F.Cu at (113.8, 148.4)
- added REF**: MountingHole_3.2mm_M3, MountingHole:MountingHole_3.2mm_M3, F.Cu at (113.8, 25.9)
- moved REF** 7.28 mm to (129.4, 111.3)
- moved REF** 6.56 mm to (129.4, 86.7)
- moved REF** 6.56 mm to (129.4, 75.7)
- moved REF** 6.56 mm to (129.4, 64.7)
- moved REF** 6.56 mm to (121.3, 130.4)
- moved REF** 6.56 mm to (113.3, 64.7)
- moved REF** 6.56 mm to (113.3, 86.7)
- moved REF** 6.56 mm to (114.1, 36.7)
- moved REF** 6.56 mm to (113.3, 75.7)
- moved REF** 6.56 mm to (128.6, 36.7)
- moved REF** 6.56 mm to (113.4, 110.8)
- moved REF** 6.56 mm to (113.3, 56.2)
- moved REF** 6.56 mm to (129.4, 56.2)
- moved REF** 6.54 mm to (121.3, 110.7)
